Commit message: MAR Quadrupled Robot - ROS2 Humble Gazebo simulation with keyboard teleop and IK control

File: Quadra_gazebo_sim/description/consts.xacro (robot description, xacro)
@@ -1,5 +1,4 @@
 <?xml version="1.0"?>
 <robot name="consts" xmlns:xacro="http://www.ros.org/wiki/xacro">
-    <!-- joint limits -->
     <xacro:property name="hip_low_limit"  value="-1.57"/>
     <xacro:property name="hip_up_limit"   value="1.57"/>
@@ -10,5 +9,4 @@
     <xacro:property name="velocity"       value="1"/>
     <xacro:property name="effort"         value="10"/>
-    <!-- joint dynamics -->
     <xacro:property name="use_dynamics" value="true"/>
     <xacro:macro name="hip_joint_dynamics">
@@ -21,5 +19,4 @@
         <dynamics damping="0.01" friction="10000"/>
     </xacro:macro>
-    <!-- configure inertia -->
     <xacro:property name="body_mass" value="3"/>
     <xacro:property name="body_inertia_x_len" value="0.28"/>
@@ -38,5 +35,4 @@
     <xacro:property name="lleg_inertia_y_len" value="0.001"/>
     <xacro:property name="lleg_inertia_z_len" value="0.005"/>
-    <!-- feet -->
     <xacro:property name="foot_mass" value="0.1"/>
     <xacro:property name="foot_radius" value="0.02"/>

File: Quadra_gazebo_sim/description/gazebo_ros2_control_plugin.xacro (robot description, xacro)
@@ -1,12 +1,4 @@
 <?xml version="1.0"?>
 <robot xmlns:xacro="http://www.ros.org/wiki/xacro">
-<!-- ************* JOINT CONTROLLER GAZEBO PLUGIN ************** -->
-    <!--
-    _____________________________________________________________________
-        include this file into: /description/hyperdog.urdf.xacro
-        using following line:
-                    <xacro:include filename="gazebo_ros2_control_plugin.xacro" />
-    _____________________________________________________________________ -->
-    <!-- CONFIGURE JOINTS OF THE ROBOT -->
     <ros2_control name="GazeboSystem" type="System">
         <hardware>
@@ -146,8 +138,9 @@
         </joint>
     </ros2_control>
-    <!--  CONFIGURE THE GAZEBO PLUGIN -->
     <gazebo>
         <plugin filename="libgazebo_ros2_control.so" name="gazebo_ros2_control">
           <parameters>$(find hyperdog_gazebo_sim)/config/hyperdog_joint_controller.yaml</parameters>
+          <robot_param>robot_description</robot_param>
+          <robot_param_node>robot_state_publisher</robot_param_node>
         </plugin>
     </gazebo>

File: Quadra_gazebo_sim/description/hyperdog.urdf.xacro (robot description, xacro)
@@ -1,9 +1,6 @@
 <?xml version="1.0"?>
 <robot xmlns:xacro="http://www.ros.org/wiki/xacro"  name="hyperdog">
-    <!-- ***************  CONFIGURE ROBOT"S LINKS  *******************-->
     <xacro:include filename="hyperdog_urdf_links.xacro" />
-    <!-- ***************  CONFIGURE ROBOT"S JOINTS  *******************-->
     <xacro:include filename="hyperdog_urdf_joints.xacro" />
-    <!-- ****************   INCLUDES OTHER FILES  ******************* -->
     <xacro:include filename="gazebo_ros2_control_plugin.xacro" />
     <xacro:include filename="hyperdog_gazebo.xacro" />

File: Quadra_gazebo_sim/description/hyperdog_gazebo.xacro (robot description, xacro)
@@ -1,13 +1,4 @@
 <?xml version="1.0"?>
 <robot xmlns:xacro="http://www.ros.org/wiki/xacro">
-<!--
-    _____________________________________________________________________
-        include this file into: /description/hyperdog.urdf.xacro
-        using following line:
-                    <xacro:include filename="hyperdog_gazebo.xacro" />
-    _____________________________________________________________________
-    * Gazebo is unable to use the same <material> tags that are already in the URDF (that RViz uses).
-    Instead, we need to add gazebo tags for our links that refer to Gazebo materials
--->
     <xacro:include filename="physics.xacro" />
     <xacro:macro name="gz_hip">
@@ -28,6 +19,4 @@
         <self_collide>1</self_collide>
         <material>Gazebo/Orange</material>
-        <!-- <implicitSpringDamper>1</implicitSpringDamper>
-        <springStiffness>100</springStiffness> -->
     </xacro:macro>
     <xacro:macro name="gz_lleg">
@@ -41,6 +30,4 @@
         <material>Gazebo/DarkYellow</material>
         <minDepth>0.001</minDepth>
-        <!-- <implicitSpringDamper>1</implicitSpringDamper>
-        <springStiffness>100</springStiffness> -->
     </xacro:macro>
     <xacro:macro name="gz_foot">
@@ -57,14 +44,10 @@
         <material>Gazebo/DarkGrey</material>
     </xacro:macro>
-    <!-- body -->
     <gazebo reference="base_link">
         <mu1>0.05</mu1>
         <mu2>0.05</mu2>
-        <!-- <kp>1000000.0</kp>
-        <kd>1.0</kd> -->
         <maxVel>0.01</maxVel>
         <material>Gazebo/DarkGrey  </material>
     </gazebo>
-    <!-- hip -->
     <gazebo reference="FR_hip_link">
         <xacro:gz_hip></xacro:gz_hip>
@@ -79,5 +62,4 @@
         <xacro:gz_hip></xacro:gz_hip>
     </gazebo>
-    <!-- uleg -->
     <gazebo reference="FR_uleg_link">
         <xacro:gz_uleg></xacro:gz_uleg>
@@ -92,5 +74,4 @@
         <xacro:gz_uleg></xacro:gz_uleg>
     </gazebo>
-    <!-- lleg -->
     <gazebo reference="FR_lleg_link">
         <xacro:gz_lleg></xacro:gz_lleg>
@@ -105,5 +86,4 @@
         <xacro:gz_lleg></xacro:gz_lleg>
     </gazebo>
-    <!-- feet -->
     <gazebo reference="FR_foot">
         <xacro:gz_foot></xacro:gz_foot>

File: Quadra_gazebo_sim/description/hyperdog_urdf_joints.xacro (robot description, xacro)
@@ -1,14 +1,7 @@
 <?xml version="1.0"?>
 <robot xmlns:xacro="http://www.ros.org/wiki/xacro">
-<!--
-    _____________________________________________________________________
-        include this file into: /description/hyperdog.urdf.xacro
-        using following line:
-                    <xacro:include filename="hyperdog_urdf_joints.xacro" />
-    _____________________________________________________________________ -->
     <xacro:include filename="consts.xacro" />
-    <!-- Limits -->
     <xacro:macro name="hip_limits">
-        <limit lower="${hip_low_limit}" upper="${hip_up_limit}" velocity="${velocity}" effort="${effort}"/> <!-- effort = 7 -->
+        <limit lower="${hip_low_limit}" upper="${hip_up_limit}" velocity="${velocity}" effort="${effort}"/>
     </xacro:macro>
     <xacro:macro name="uleg_limits">
@@ -18,10 +11,8 @@
         <limit lower="${lleg_low_limit}" upper="${lleg_up_limit}" velocity="${velocity}" effort="${effort}"/>
     </xacro:macro>
-    <!-- ******** Inertial-base joint ********** -->
     <joint name="inertial_joint" type="fixed">
         <parent link="base_link"/>
         <child link="inertial_link"/>
     </joint>
-    <!-- *********  FR_hip joint ********* -->
     <joint name="FR_hip_joint" type="revolute">
         <axis xyz="-1 0 0"/>
@@ -34,5 +25,4 @@
         </xacro:if>
     </joint>
-    <!-- *********  FL_hip  ********* -->
     <joint name="FL_hip_joint" type="revolute">
         <axis xyz="1 0 0"/>
@@ -45,5 +35,4 @@
         </xacro:if>
     </joint>
-    <!-- *********  BR_hip  ********* -->
     <joint name="BR_hip_joint" type="revolute">
         <axis xyz="-1 0 0"/>
@@ -56,5 +45,4 @@
         </xacro:if>
     </joint>
-    <!-- *********  BL_hip  ********* -->
     <joint name="BL_hip_joint" type="revolute">
         <axis xyz="1 0 0"/>
@@ -67,5 +55,4 @@
         </xacro:if>
     </joint>
-    <!-- *********  FR_uleg joint ********* -->
     <joint name="FR_uleg_joint" type="revolute">
         <axis xyz="0 -1 0"/>
@@ -78,5 +65,4 @@
         </xacro:if>
     </joint>
-    <!-- *********  FL_uleg  ********* -->
     <joint name="FL_uleg_joint" type="revolute">
         <axis xyz="0 -1 0"/>
@@ -89,5 +75,4 @@
         </xacro:if>
     </joint>
-    <!-- *********  BR_uleg  ********* -->
     <joint name="BR_uleg_joint" type="revolute">
         <axis xyz="0 -1 0"/>
@@ -100,5 +85,4 @@
         </xacro:if>
     </joint>
-    <!-- *********  BL_uleg  ********* -->
     <joint name="BL_uleg_joint" type="revolute">
         <axis xyz="0 -1 0"/>
@@ -111,5 +95,4 @@
         </xacro:if>
     </joint>
-    <!-- *********  FR_lleg  ********* -->
     <joint name="FR_lleg_joint" type="revolute">
         <axis xyz="0 1 0"/>
@@ -122,5 +105,4 @@
         </xacro:if>
     </joint>
-    <!-- *********  FL_lleg  ********* -->
     <joint name="FL_lleg_joint" type="revolute">
         <axis xyz="0 1 0"/>
@@ -133,5 +115,4 @@
         </xacro:if>
     </joint>
-    <!-- *********  BR_lleg  ********* -->
     <joint name="BR_lleg_joint" type="revolute">
         <origin xyz="-0.15 0 0" rpy="0 0.0 0"/>
@@ -144,5 +125,4 @@
         </xacro:if>
     </joint>
-    <!-- *********  BL_lleg  ********* -->
     <joint name="BL_lleg_joint" type="revolute">
         <axis xyz="0 1 0"/>
@@ -155,5 +135,4 @@
         </xacro:if>
     </joint>
-     <!-- *********  FR_FOOT  ********* -->
      <joint name="FR_foot_fixed" type="fixed">
         <origin rpy="0 0 0" xyz="0.14 0 0"/>
@@ -161,5 +140,4 @@
         <child link="FR_foot"/>
       </joint>
-     <!-- *********  FL_FOOT  ********* -->
      <joint name="FL_foot_fixed" type="fixed">
         <origin rpy="0 0 0" xyz="0.14 0 0"/>
@@ -167,5 +145,4 @@
         <child link="FL_foot"/>
       </joint>
-     <!-- *********  BR_FOOT  ********* -->
      <joint name="BR_foot_fixed" type="fixed">
         <origin rpy="0 0 0" xyz="0.14 0 0"/>
@@ -173,5 +150,4 @@
         <child link="BR_foot"/>
       </joint>
-    <!-- *********  BL_FOOT  ********* -->
     <joint name="BL_foot_fixed" type="fixed">
         <origin rpy="0 0 0" xyz="0.14 0 0"/>

File: Quadra_gazebo_sim/description/hyperdog_urdf_links.xacro (robot description, xacro)
@@ -1,15 +1,6 @@
 <?xml version="1.0"?>
 <robot xmlns:xacro="http://www.ros.org/wiki/xacro">
-<!--
-    * Autor: nipun.dhananjaya@gmail.com
-    * Date:  13.03.2023
-    _____________________________________________________________________
-        include this file into: /description/hyperdog.urdf.xacro
-        using following line:
-                    <xacro:include filename="hyperdog_urdf_links.xacro" />
-    _____________________________________________________________________ -->
     <xacro:include filename="consts.xacro" />
     <xacro:include filename="physics.xacro" />
-    <!-- load meshes -->
     <xacro:macro name="body_mesh">
         <mesh filename="file://$(find hyperdog_gazebo_sim)/meshes/body.stl" scale="0.001 0.001 0.001"/>
@@ -30,12 +21,10 @@
         <mesh filename="file://$(find hyperdog_gazebo_sim)/meshes/LLEG.stl" scale="0.001 0.001 0.001"/>
     </xacro:macro>
-    <!-- *********** Inertial link *********** -->
     <link name="inertial_link">
         <xacro:inertial_body></xacro:inertial_body>
     </link>
-    <!-- *********** base link *********** -->
     <link name="base_link">
         <visual>
-            <origin xyz="0 0 0" rpy="0 0 0"/>
+            <origin xyz="0 0 0" rpy="3.14159 0 0"/>
             <geometry>
                 <xacro:body_mesh></xacro:body_mesh>
@@ -52,6 +41,4 @@
         </collision>
     </link>
-    <!-- !!!!!!!!!!!!!!!!!!!!!!! HIPS !!!!!!!!!!!!!!!!!!!!!!!!!!!! -->
-    <!-- *********** FR_hip *********** -->
     <link name="FR_hip_link">
         <visual>
@@ -72,5 +59,4 @@
         <xacro:inertial_right_hip></xacro:inertial_right_hip>
     </link>
-    <!-- *********** FL_hip ********** -->
     <link name="FL_hip_link">
         <visual>
@@ -91,5 +77,4 @@
         <xacro:inertial_left_hip></xacro:inertial_left_hip>
     </link>
-    <!-- *********** BR_hip ********** -->
     <link name="BR_hip_link">
         <visual>
@@ -110,5 +95,4 @@
         <xacro:inertial_right_hip></xacro:inertial_right_hip>
     </link>
-    <!-- *********** BL_hip ********** -->
     <link name="BL_hip_link">
         <visual>
@@ -129,6 +113,4 @@
         <xacro:inertial_left_hip></xacro:inertial_left_hip>
     </link>
-    <!-- !!!!!!!!!!!!!!!!!!!!!!! ULEGs !!!!!!!!!!!!!!!!!!!!!!!!!!!! -->
-    <!-- *********** FR_uleg ********** -->
     <link name="FR_uleg_link">
         <visual>
@@ -149,5 +131,4 @@
         <xacro:inertial_right_uleg></xacro:inertial_right_uleg>
     </link>
-    <!-- *********** FL_uleg ********** -->
     <link name="FL_uleg_link">
         <visual>
@@ -168,5 +149,4 @@
         <xacro:inertial_left_uleg></xacro:inertial_left_uleg>
     </link>
-    <!-- *********** BR_uleg ********** -->
     <link name="BR_uleg_link">
         <visual>
@@ -187,5 +167,4 @@
         <xacro:inertial_right_uleg></xacro:inertial_right_uleg>
     </link>
-    <!-- *********** BL_uleg ********** -->
     <link name="BL_uleg_link">
         <visual>
@@ -206,6 +185,4 @@
         <xacro:inertial_left_uleg></xacro:inertial_left_uleg>
     </link>
-    <!-- !!!!!!!!!!!!!!!!!!!!!!! LLEGs !!!!!!!!!!!!!!!!!!!!!!!!!!!! -->
-    <!-- *********** FR_lleg ********** -->
     <link name="FR_lleg_link">
         <visual>
@@ -226,5 +203,4 @@
         <xacro:inertial_right_lleg></xacro:inertial_right_lleg>
     </link>
-    <!-- *********** FL_lleg ********** -->
     <link name="FL_lleg_link">
         <visual>
@@ -245,5 +221,4 @@
         <xacro:inertial_left_lleg></xacro:inertial_left_lleg>
     </link>
-      <!-- *********** BR_lleg ********** -->
     <link name="BR_lleg_link">
         <visual>
@@ -264,5 +239,4 @@
         <xacro:inertial_right_lleg></xacro:inertial_right_lleg>
     </link>
-    <!-- *********** BL_lleg ********** -->
     <link name="BL_lleg_link">
         <visual>
@@ -283,6 +257,4 @@
         <xacro:inertial_left_lleg></xacro:inertial_left_lleg>
     </link>
-    <!-- !!!!!!!!!!!!!!!!!!!!!!! FEET !!!!!!!!!!!!!!!!!!!!!!!!!!!! -->
-    <!-- *********** FL FOOT ********** -->
     <link name="FL_foot">
         <visual>
@@ -310,5 +282,4 @@
         <xacro:inertial_foot></xacro:inertial_foot>
       </link>
-    <!-- *********** FR FOOT ********** -->
     <link name="FR_foot">
         <visual>
@@ -336,5 +307,4 @@
         <xacro:inertial_foot></xacro:inertial_foot>
       </link>
-    <!-- *********** BR FOOT ********** -->
     <link name="BR_foot">
         <visual>
@@ -362,5 +332,4 @@
         <xacro:inertial_foot></xacro:inertial_foot>
       </link>
-    <!-- *********** BL FOOT ********** -->
     <link name="BL_foot">
         <visual>

File: Quadra_gazebo_sim/description/physics.xacro (robot description, xacro)
@@ -2,13 +2,11 @@
 <robot xmlns:xacro="http://www.ros.org/wiki/xacro" >
     <xacro:include filename="consts.xacro" />
-    <!--  BODY -->
     <xacro:macro name="inertial_body">
         <inertial>
-            <origin xyz="-0.006 0.00633 0.00214" rpy="0 0 0"/> <!-- 0.006, -0.000233, 0.00214 -->
+            <origin xyz="-0.006 0.00633 0.00214" rpy="0 0 0"/>
             <mass value="${body_mass}" />
             <inertia  ixx="0.011396658109874464" ixy="0" ixz="0" iyy="0.05486450023370329" iyz="0" izz="0.06098759357764758" />
         </inertial>
     </xacro:macro>
-    <!-- HIP -->
     <xacro:macro name="inertial_right_hip">
         <inertial>
@@ -25,5 +23,4 @@
         </inertial>
     </xacro:macro>
-    <!-- ULEG -->
     <xacro:macro name="inertial_right_uleg">
         <inertial>
@@ -40,5 +37,4 @@
         </inertial>
     </xacro:macro>
-    <!-- LLEG -->
     <xacro:macro name="inertial_right_lleg">
         <inertial>
@@ -55,5 +51,4 @@
         </inertial>
     </xacro:macro>
-    <!-- FOOT -->
     <xacro:macro name="inertial_foot">
         <inertial>
@@ -65,4 +60,3 @@
         </inertial>
     </xacro:macro>
-    <!-- ************************************************************************************************** -->
 </robot>
